File: adapter.kicad_sch (KiCad schematic)
At the start: 13 parts, among them U1 nRF9161-SIXX

Commit message: feat: add gps amplifier
Parts:
- added C10, C11, C12: 39pF, symbol Device:C
- added C13: 33nF, symbol Device:C
- added C14: 1nF, symbol Device:C
- added L1: 68nH, symbol Device:L
- added L2: 8.2nH, symbol Device:L
- added N1: ~, symbol tracker_symbols_library:BGA524N6
Connections:
- net GND: now also C12.1, N1.1 (GND), N1.4 (GNDRF)
- net at U1.67 (GPS): now also C10.2
- net at U1.93 (COEX0): now also N1.6 (PON)
- new net: C13.2, N1.2 (VCC)
- new net: C11.1, N1.3 (AO)
- new net: C10.1, C11.2, L1.1
- new net: C14.1, L2.2
- new net: L2.1, N1.5 (AI)
- new net VDD_LNA: C12.2, C13.1, L1.2
